File: eagle/RF Glow Stick/RF Glow Stick.sch (EAGLE design)
At the start: 8 parts, among them J1 GROVE-4P-2.0

Commit message: Fixed flawed board design. The LED connector needs to be in the middle to clear the PCB holding ledges and to have maximum clearance for round handles. Also reduced the side of the board from 5.08cm long (2 inches) to 4.99cm for cheaper Fusion PCB pricing.
Changed lines of the file:
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@@
 <wire x1="7.62" y1="114.3" x2="7.62" y2="73.66" width="0.1524" layer="91"/>
 <pinref part="R1" gate="G$1" pin="1"/>
+<junction x="7.62" y="73.66"/>
 </segment>
 </net>

Commit message: Updated board to be compatible with milling fabrication (e.g. a CNC mill with an engraving tool for isolation routing). However, actual isolution routed board is nonfunctional because the design relies upon through-plated holes to connect the top and bottom traces.
Changed lines of the file:
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@@
 <?xml version="1.0" encoding="utf-8"?>
 <!DOCTYPE eagle SYSTEM "eagle.dtd">
-<eagle version="6.5.0">
+<eagle version="7.1.0">
 <drawing>
 <settings>
@@
 <part name="FRAME1" library="frames" deviceset="LETTER_P" device=""/>
 <part name="GND1" library="supply1" deviceset="GND" device=""/>
-<part name="S1" library="switch" deviceset="TL32PO" device="" value=""/>
+<part name="S1" library="switch" deviceset="TL32PO" device="" value="TL32PO"/>
 <part name="G1" library="battery" deviceset="AB9V" device="" value=""/>
 <part name="J1" library="My Library" deviceset="GROVE-4P-2.0" device=""/>
@@
 </sheet>
 </sheets>
+<errors>
+</errors>
 </schematic>
 </drawing>
